Commit message: TB add missing models,  tweek failscale/dyn just a little to improve sensitivity since they will hae ~20 false before true..

File: cartpolepp/models/ground_cart.urdf (robot description, URDF)
Before this commit: robot ground, 3 links, 2 joints
Links:
- link ground: geometry visual box size=0.1 0.1 0.3
- link pole: geometry collision cylinder length=1.0 radius=0.03; visual cylinder length=1.0 radius=0.03
Joints:
- joint pole_to_cart: origin xyz=0.0 0.0 0.2 -> xyz=0.0 0.0 0.2 rpy=0 0 0
